Commit message: feat: add front cam to the model

File: go2_robot_sdk/urdf/go2.urdf (robot description, URDF)
Before this commit: robot go2, 29 links, 28 joints
Links:
- added link front_camera; collision cylinder length=0.09 radius=0.05; visual cylinder length=0.01 radius=0.01
Joints:
- added joint front_camera_joint: type fixed, parent Head_upper, child front_camera, origin xyz=0.045 0 0.03 rpy=-1.5708 0 -1.5708, axis 0 0 0

Commit message: added slam_toolbox + twist mux

File: go2_robot_sdk/urdf/go2.urdf (robot description, URDF)
Before this commit: robot go2, 29 links, 28 joints
Links:
- added link base_footprint
- added link map
- added link odom
Joints:
- added joint base_footprint_joint: type fixed, parent base, child base_footprint, origin xyz=0 0 0 rpy=0 0 0
- added joint map_joint: type fixed, parent odom, child map, origin xyz=0 0 0 rpy=0 0 0
- added joint odom_joint: type fixed, parent odom, child base, origin xyz=0 0 0 rpy=0 0 0

Commit message: some minor fix

File: go2_robot_sdk/urdf/go2.urdf (robot description, URDF)
Before this commit: robot go2, 31 links, 30 joints
Links:
- removed link base
- added link base_link, mass 6.921; collision box size=0.3762 0.0935 0.114; visual mesh filename=package://go2_robot_sdk/dae/base.dae
Joints:
- joint FL_hip_joint: parent base -> base_link
- joint FR_hip_joint: parent base -> base_link
- joint Head_upper_joint: parent base -> base_link
- joint RL_hip_joint: parent base -> base_link
- joint RR_hip_joint: parent base -> base_link
- joint imu_joint: parent base -> base_link
- joint map_joint: child map -> odom; parent odom -> map
- joint odom_joint: child base -> base_link
- joint radar_joint: parent base -> base_link

File: go2_robot_sdk/urdf/go2_on_steroids.urdf (robot description, URDF)
Before this commit: robot go2, 33 links, 32 joints
Links:
- removed link base
- added link base_link, mass 6.921; collision box size=0.3762 0.0935 0.114; visual mesh filename=package://go2_robot_sdk/meshes/base_link.STL
Joints:
- joint FL_hip_joint: parent base -> base_link
- joint FR_hip_joint: parent base -> base_link
- joint Head_upper_joint: parent base -> base_link
- joint RL_hip_joint: parent base -> base_link
- joint RR_hip_joint: parent base -> base_link
- joint front_d_camera_joint: parent base -> base_link
- joint imu_joint: parent base -> base_link
- joint left_d_camera_joint: parent base -> base_link
- joint lidar_joint: parent base -> base_link
- joint radar_joint: parent base -> base_link
- joint right_d_camera_joint: parent base -> base_link

Commit message: fix: rotate optical frame to ROS2 convention

File: go2_robot_sdk/urdf/go2.urdf (robot description, URDF)
Before this commit: robot go2, 33 links, 32 joints
Joints:
- joint front_camera_joint: origin xyz=0.045 0 0.03 rpy=-1.5708 0 -1.5708 -> xyz=0.045 0 0.03 rpy=1.5708 0 1.5708
